File: kicad_template.kicad_sch (KiCad schematic)
At the start: 0 parts

Commit message: Update page setup
Other:
- company: Ontario Tech Racing -> Daniel Jeon
Changed lines of the file:
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@@
 	(title_block
 		(title "Template")
-		(company "Ontario Tech Racing")
+		(company "Daniel Jeon")
 	)
 	(sheet_instances
